File: LIN-Controller.sch (KiCad schematic (older format))
At the start: 52 parts, among them CON1 BARREL_JACK, J1 SWD_HEADER, J2 1881451_LIN, SW1 GP12MCBE, SW2 THUMBWHEEL, SW3 TL9210, SW4 TL9210, SW5 TL9210, SW6 TL9210, U1 2SC5662, U2 SAMC21E-A, U3 TPS7133QD, U4 2SC5662, U5 2SC5662, U6 2SC5662, U7 ATA663211

Commit message: Added files via upload
Parts:
- removed C1, C2, C3: 0.1u, ~, symbol C
- removed D1, D3, D4, D5: 7_SEGMENT_DISPLAY, symbol 7_SEGMENT_DISPLAY
- removed D2: XZMYR155W, symbol XZMYR155W
- removed R1, R11, R17, R2, R3, R4, R5, R6, R7: 200, ~, symbol R
- removed R10, R9: 10K, ~, symbol R
- removed R12, R13, R14, R22, R23, R24, R25: 4K7, ~, symbol R
- removed R8: 22R, ~, symbol R
- removed SW1: GP12MCBE, symbol GP12MCBE
- removed SW2: THUMBWHEEL, ~, symbol THUMBWHEEL
- removed SW5, SW6: TL9210, symbol TL9210
- removed U1: 2SC5662, symbol 2SC5662
- removed U2: SAMC21E-A, TQFP32, symbol SAMC21E-A
- removed U3: TPS7133QD, SO-8, symbol TPS7133QD
- added C1: 47u, ~, symbol C-RESCUE-LIN-Controller1.1
- added C2, C4, C5: 0.1u, ~, symbol C-RESCUE-LIN-Controller1.1
- added C3: 100u, ~, symbol C-RESCUE-LIN-Controller1.1
- added D1, D3, D4, D5: HDSM-283L, symbol HDSM-283L
- added D2: 1N5819, symbol 1N5819
- added L1: 33u, ~, symbol INDUCTOR_SMALL
- added R1, R6: 10K, ~, symbol R-RESCUE-LIN-Controller1.1
- added R2, R3, R4, R5: 330R, ~, symbol R-RESCUE-LIN-Controller1.1
- added R7: 22R, ~, symbol R-RESCUE-LIN-Controller1.1
- added SW1, SW2: TL9210, symbol TL9210
- added SW5: TSWA3NCD23LFS_, symbol TSWA3NCD23LFS_
- added U1: SAMC21E-A, TQFP32, symbol SAMC21E-A
- added U2: 2SC5662, ~, symbol 2SC5662
- added U3: LM2675, ~, symbol LM2675
- C7, C8, C9: symbol C -> C-RESCUE-LIN-Controller1.1
- J1, U4, U5, U6: footprint (none) -> ~
- R15, R16, R19, R20, R21: symbol R -> R-RESCUE-LIN-Controller1.1
Connections:
- net Vcc is gone; now on net 3V3: J1.1 (VTref), R20.1
- net 3V3: now also C3.1, L1.2, R1.1, R6.1, U3.4 (FS)
- net GND: now also SW3.1, SW4.1, C1.2, C3.2, C4.2, C5.2, D2.1, SW1.1, SW2.1, SW5.4 (COM), U1.10 (GND), U1.28 (GND), U2.2 (E), U3.6 (GND); no longer SW3.2, SW4.2
- net VsLIN: now also D6.3, C1.1, U3.7 (Vin)
- net at U6.3 (C): now also D5.3 (CC)
- net at U5.3 (C): now also D4.3 (CC)
- net at U4.3 (C): now also D3.3 (CC)
- net at U4.1 (B): now also R3.2
- net at U5.1 (B): now also R4.2
- net at J1.10 (nRESET): now also U1.26 (~RESET~)
- net at U6.1 (B): now also R5.2
- net at J1.4 (SWDCLK): now also R6.2, U1.31 (GCLKIO0/SWCLK/TC1WO0/SERCOM1P2/PA30)
- net EN: now reaches U7.2 (EN)
- net EN: now also U1.5 (TC0WO0/SERCOM0P0/Y2/AIN0/AIN4/VREFB/PA04)
- net TXD: now reaches U7.4 (TXD)
- net TXD: now also U1.6 (TC0W01/SERCOM0P1/Y3/AIN1/AIN5/PA05)
- net RXD: now reaches R20.2, U7.1 (RXD)
- net RXD: now also U1.7 (TC1WO0/SERCOM0P2/Y4/AIN2/AIN6/PA06)
- net at J2.1: now also D6.2
- net at D6.1: now also R15.2
- net at J1.2 (SWDIO): now also R1.2, R7.2
- new net: C5.1, U1.29 (VDDCORE)
- new net: C4.1, U1.30 (VDDIN)
- new net: R7.1, U1.32 (SWDIO/TC1WO1/SERCOM1P3/PA31)
- new net: R2.2, U2.1 (B)
- new net: D1.3 (CC), U2.3 (C)
- new net: C2.1, U3.1 (CB)
- new net: C2.2, D2.2, L1.1, U3.8 (VSW)
- new net DIS'.': D1.7 (D2), D3.7 (D2), D4.7 (D2), D5.7 (D2), U1.24 (TC5WO1/SERCOM5P3/SERCOM3P3/PA25)
- new net DIS'a': D1.6 ('b'), D3.6 ('b'), D4.6 ('b'), D5.6 ('b'), U1.23 (TC5WO0/SERCOM5P2/SERCOM3P2/PA24)
- new net DIS'b': D1.5 ('a'), D3.5 ('a'), D4.5 ('a'), D5.5 ('a'), U1.22 (GCLKIO7/TC4WO1/SERCOM5P1/SERCOM3P1/X11/PA23)
- new net DIS'c': D1.8 ('c'), D3.8 ('c'), D4.8 ('c'), D5.8 ('c'), U1.21 (GCLKIO6/TC4WO0/SERCOM5P0/SERCOM3P0/X10/PA22)
- new net DIS'd': D1.10 ('d'), D3.10 ('d'), D4.10 ('d'), D5.10 ('d'), U1.20 (ACCMP1/TC3WO1/SERCOM3P3/SERCOM1P3/X7/PA19)
- new net DIS'e': D1.11 ('e'), D3.11 ('e'), D4.11 ('e'), D5.11 ('e'), U1.19 (ACCMP0/TC3WO0/SERCOM3P2/SERCOM1P2/X6/PA18)
- new net DIS'f': D1.3 (CC), D3.3 (CC), D4.3 (CC), D5.3 (CC), U1.18 (GCLKIO3/TC2WO1/SERCOM3P1/SERCOM1P1/X5/PA17)
- new net DIS'g': D1.1 ('g'), D3.1 ('g'), D4.1 ('g'), D5.1 ('g'), U1.17 (GCLKIO2/TC2WO0/SERCOM3P0/SERCOM1P0/X4/PA16)
- new net DS0: R5.1, U1.27 (GCLKIO0/PA28)
- new net DS1: R4.1, U1.25 (GCLKIO0/PA27)
- new net DS2: R3.1, U1.16 (XOUT/GCLKIO1/TC3WO1/SERCOM4P3/SERCOM2P3/PA15)
- new net DS3: R2.1, U1.15 (XIN/GCLKIO0/TC3WO0/SERCOM4P2/SERCOM2P2/PA14)
- new net PB0: SW1.2, U1.14 (GCLKIO5/TC1WO1/SERCOM2P3/SERCOM0P3/X3/AIN19/PA11)
- new net PB1: SW2.2, U1.13 (GCLKIO4/TC1WO0/SERCOM2P2/SERCOM0P2/X2/AIN18/PA10)
- new net PB2: SW3.2, U1.12 (TC0WO1/SERCOM2P1/SERCOM0P1/X1/AIN17/PA09)
- new net PB3: SW4.2, U1.11 (TC0WO0/SERCOM2P0/SERCOM0P0/X0/AIN16/NMI/PA08)
- new net TWA: SW5.1 (A), U1.2 (XOUT32/TC2WO1/SERCOM1P1/PA01)
- new net TWB: SW5.2 (B), U1.3 (VOUT/Y0/AIN0/PA02)
- new net TWC: SW5.3 (NO), U1.1 (XIN32/TC2WO0/SERCOM1P0/PA00)
Other:
- note removed: "Display"
- note removed: "Input Buttons"
- note removed: "LIN Bus Interface"
- note removed: "LIN Interfacing\nSERCOMOP0 Pin 5 EN\nSERCOMOP1 Pin6 TXD\nSERCOMOP2 Pin7 RXD\n\nDISPLAYS\nPA16 Pin17 Element 'g'\nPA17 Pin18 Element 'f'\nPA18 Pin19 Element 'e'\nPA19 Pin20 Element 'd'\nPA20 Pin21 Element 'c'\nPA21 Pin22 Element 'b'\nPA22 Pin23 Element 'a'\nPA23 Pin24 Decimal Point\nPA14 Pin15 1000's display select\nPA15 Pin16 100's display select\nPA27 Pin26 10's display select\nPA28 Pin27 1's di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"
- note removed: "Power Supply"
- note removed: "Programming Connector"
- note removed: "SAMC21 I/O Port Allocations"
- note removed: "Thumb-wheel and Button"
- moved on the sheet: C7, C8, C9, CON1, D6, J2, R15, R16, R19, R20, R21, U7
